Commit message: Update ultrasound.urdf.xacro

File: src/raskar_urdf/urdf/ultrasound.urdf.xacro (robot description, xacro)
@@ -49,5 +49,5 @@
       <parent link="${parent}"/>
       <child link="${fb}_${cnc}_${lr}_ultrasound"/>
-      <origin xyz="${translateX * base_x_origin_to_ultrasound_origin} ${translateY * base_y_origin_to_ultrasound_origin} ${translateZ * base_z_origin_to_ultrasound_origin}" rpy="0 0 ${rotateTheta*Pi/180}"/>
+      <origin xyz="${translateX * base_x_origin_to_ultrasound_origin} ${translateY * base_y_origin_to_ultrasound_origin} ${base_z_origin_to_ultrasound_origin + translateZ}" rpy="0 0 ${rotateTheta*Pi/180}"/>
     </joint>
     <!-- Transmission is important to link the joints and the controller -->
