Commit message: Update gazebo sim static links

File: src/raskar_urdf/urdf/lidar.urdf.xacro (robot description, xacro)
@@ -35,11 +35,7 @@
     </link>
     <gazebo reference="${fb}_${cnc}_${lrc}_lidar">
-      <mu1 value="1.0"/>
-      <mu2 value="1.0"/>
-      <kp  value="10000000.0" />
-      <kd  value="1.0" />
-      <fdir1 value="1 0 0"/>
-      <material>Gazebo/Grey</material>
-      <turnGravityOff>false</turnGravityOff>
+      <static>true</static>
+      <material>Gazebo/Black</material>
+      <turnGravityOff>true</turnGravityOff>
     </gazebo>
     <joint name="${fb}_${cnc}_${lrc}_lidar_joint" type="fixed">
@@ -48,15 +44,4 @@
       <origin xyz="${translateX * base_x_origin_to_lidar_origin} ${translateY * base_y_origin_to_lidar_origin} ${base_z_origin_to_lidar_origin + (thickness_lidar/2) + translateZ}" rpy="0 0 0" />
     </joint>
-    <!-- Transmission is important to link the joints and the controller -->
-    <transmission name="${fb}_${cnc}_${lrc}_lidar_joint_trans">
-      <type>transmission_interface/SimpleTransmission</type>
-      <joint name="${fb}_${cnc}_${lrc}_lidar_joint">
-        <hardwareInterface>EffortJointInterface</hardwareInterface>
-      </joint>
-      <actuator name="${fb}_${cnc}_${lrc}_lidar_joint_motor">
-        <hardwareInterface>EffortJointInterface</hardwareInterface>
-        <mechanicalReduction>1</mechanicalReduction>
-      </actuator>
-    </transmission>
   </xacro:macro>
 </robot>

File: src/raskar_urdf/urdf/raskar_gazebo.xacro (robot description, xacro)
@@ -14,4 +14,6 @@
   <xacro:property name="thickness_lidar" value="0.045" /> <!-- Thickness of wheel -->
   <xacro:property name="safety_offset"   value="1.25"  /> <!-- Percentage safety  -->
+  <xacro:property name="floor_clearance" value="0.0350"/> <!-- Floor clearance    -->
+  <xacro:property name="model_offset"    value="0.0127"/> <!-- Floor clearance    -->
   <!-- Gazebo initializer -->
   <!-- Import all Gazebo-customization elements, including Gazebo colors -->
@@ -24,4 +26,5 @@
   <!-- Import Sensors -->
   <xacro:include filename="$(find raskar_urdf)/urdf/ultrasound.urdf.xacro" />
+  <xacro:include filename="$(find raskar_urdf)/urdf/lidar.urdf.xacro" />
   <!-- Macro for calculating inertia of cylinder -->
   <macro name="cylinder_inertia" params="m r h">
@@ -30,8 +33,14 @@
               izz="${m*r*r/2}" />
   </macro>
+  <!-- Macro for calculating inertia of box -->
+  <macro name="box_inertia" params="m h l w">
+    <inertia  ixx="${m*(h*h+l*l)/12}" ixy = "0" ixz = "0"
+              iyy="${m*(w*w+l*l)/12}" iyz = "0"
+              izz="${m*(w*w+h*h)/12}" />
+  </macro>
   <!-- Used for fixing robot to Gazebo -->
-  <!-- link name="world"/>
+  <!-- link name="floor"/>
   <joint name="fixed" type="fixed">
-    <parent link="world"/>
+    <parent link="floor"/>
     <child link="base_footprint"/>
   </joint -->
@@ -39,5 +48,5 @@
   <!-- base_footprint is a fictitious link(frame) that is on the ground right below base_link origin -->
   <link name="base_footprint">
-    <inertial>
+    <!-- inertial>
       <mass value="0.0001" />
       <origin xyz="0 0 0" />
@@ -45,5 +54,5 @@
           iyy="0.0001" iyz="0.0"
           izz="0.0001" />
-    </inertial>
+    </inertial -->
     <visual>
         <origin xyz="0 0 0" rpy="0 0 0" />
@@ -57,5 +66,5 @@
   </gazebo>
   <joint name="base_footprint_joint" type="fixed">
-    <origin xyz="0 0 0" rpy="0 0 0" />
+    <origin xyz="0 0 ${height_body/2}" rpy="0 0 0" />
     <parent link="base_footprint"/>
     <child link="base_link" />
@@ -64,5 +73,5 @@
   <link name="base_link">
     <visual>
-      <origin rpy="1.571 0 0" xyz="0 0 -0.0127"/> <!-- Half an inch due to different wheels set up -->
+      <origin rpy="1.571 0 0" xyz="0 0 ${-height_body/2-floor_clearance-model_offset}"/> <!-- Half an inch due to different wheels set up -->
       <geometry>
         <mesh filename="package://raskar_urdf/meshes/body_parts.stl" scale="0.001 0.001 0.001" />
@@ -78,25 +87,23 @@
     </collision>
     <inertial>
-      <mass value="${mass_wheel}"/>
-      <inertia
-	  ixx="${mass_body / 12.0 * (height_body*height_body + length_body*length_body)}" ixy="0.0" ixz="0.0"
-	  iyy="${mass_body / 12.0 * (width_body*width_body + length_body*length_body)}" iyz="0.0"
-	  izz="${mass_body / 12.0 * (width_body*width_body + height_body*height_body)}"/>
+      <mass value="${mass_body}"/>
+      <origin xyz="0 0 0" />
+      <box_inertia  m="${mass_body}" h="${height_body}" l="${length_body}" w="${width_body}" />
     </inertial>
   </link>
-  <!-- Wheels definition -->
-  <wheel fb="bk" lr="right"  parent="base_link" translateX="-1" translateY="-1" translateZ="1" flipY="1"/>
-  <wheel fb="fr" lr="right"  parent="base_link" translateX="1"  translateY="-1" translateZ="1" flipY="1"/>
-  <wheel fb="fr" lr="left"   parent="base_link" translateX="1"  translateY="1"  translateZ="1" flipY="1"/>
-  <wheel fb="bk" lr="left"   parent="base_link" translateX="-1" translateY="1"  translateZ="1" flipY="1"/>
+  <!-- Wheels Definition -->
+  <wheel fb="bk" lr="left"  parent="base_link" translateX="-1" translateY="-1" translateZ="${((-height_body/2)-floor_clearance)}" flipY="1"/>
+  <wheel fb="fr" lr="left"  parent="base_link" translateX="1"  translateY="-1" translateZ="${((-height_body/2)-floor_clearance)}" flipY="1"/>
+  <wheel fb="fr" lr="right" parent="base_link" translateX="1"  translateY="1"  translateZ="${((-height_body/2)-floor_clearance)}" flipY="1"/>
+  <wheel fb="bk" lr="right" parent="base_link" translateX="-1" translateY="1"  translateZ="${((-height_body/2)-floor_clearance)}" flipY="1"/>
+  <!-- Ultrasound sensors definition -->
+  <ultrasound fb="fr" cnc="nocorner" lr="right"  parent="base_link" translateX="1" translateY="-1" translateZ="${((-height_body/2)-floor_clearance)}" flipX="90" flipY="0" flipZ="90" rotateTheta="0"/>
+  <ultrasound fb="fr" cnc="nocorner" lr="left"   parent="base_link" translateX="1" translateY="1"  translateZ="${((-height_body/2)-floor_clearance)}" flipX="90" flipY="0" flipZ="90" rotateTheta="0"/>
+  <ultrasound fb="fr" cnc="corner"   lr="right"  parent="base_link" translateX="0.8991870987"  translateY="-2.5038" translateZ="${((-height_body/2)-floor_clearance)}" flipX="90" flipY="0" flipZ="90" rotateTheta="-45"/>
+  <ultrasound fb="fr" cnc="corner"   lr="left"   parent="base_link" translateX="0.8991870987"  translateY="2.5038"  translateZ="${((-height_body/2)-floor_clearance)}" flipX="90" flipY="0" flipZ="90" rotateTheta="45"/>
+  <ultrasound fb="bk" cnc="corner"   lr="right"  parent="base_link" translateX="-0.8991870987" translateY="-2.5038" translateZ="${((-height_body/2)-floor_clearance)}" flipX="90" flipY="0" flipZ="90" rotateTheta="225"/>
+  <ultrasound fb="bk" cnc="corner"   lr="left"   parent="base_link" translateX="-0.8991870987" translateY="2.5038"  translateZ="${((-height_body/2)-floor_clearance)}" flipX="90" flipY="0" flipZ="90" rotateTheta="135"/>
   <!-- Lidar definition -->
-  <lidar fb="fr"  cnc="nocorner"   lrc="center"   parent="base_link" translateX="1" translateY="1"  translateZ="1" flipX="0" flipY="0" flipZ="0"/>
-  <!-- Ultrasound sensors Definitions -->
-  <ultrasound fb="front" cnc="nocorner" lr="right"  parent="base_link" translateX="1" translateY="-1" translateZ="1" flipX="90" flipY="0" flipZ="90"/>
-  <ultrasound fb="front" cnc="nocorner" lr="left"   parent="base_link" translateX="1" translateY="1"  translateZ="1" flipX="90" flipY="0" flipZ="90"/>
-  <ultrasound fb="front" cnc="corner"   lr="right"  parent="base_link" translateX="0.8991870987"  translateY="-2.5038" translateZ="1" flipX="90" flipY="0" flipZ="45"/>
-  <ultrasound fb="front" cnc="corner"   lr="left"   parent="base_link" translateX="0.8991870987"  translateY="2.5038"  translateZ="1" flipX="90" flipY="0" flipZ="135"/>
-  <ultrasound fb="back"  cnc="corner"   lr="right"  parent="base_link" translateX="-0.8991870987" translateY="-2.5038" translateZ="1" flipX="90" flipY="0" flipZ="315"/>
-  <ultrasound fb="back"  cnc="corner"   lr="left"   parent="base_link" translateX="-0.8991870987" translateY="2.5038"  translateZ="1" flipX="90" flipY="0" flipZ="225"/>
+  <lidar fb="fr"  cnc="nocorner"   lrc="center"  parent="base_link" translateX="1" translateY="1"  translateZ="${(-height_body/2)-floor_clearance}" flipX="0" flipY="0" flipZ="0"/>
   <!-- Motion controller -->
   <!-- Planar drive controller  -->

File: src/raskar_urdf/urdf/ultrasound.urdf.xacro (robot description, xacro)
@@ -5,5 +5,5 @@
   <property name="width_usound"     value="0.020" /> <!-- width of sensor   -->
   <property name="depth_usound"     value="0.015" /> <!-- length of sensor  -->
-  <property name="mass_usound"      value="0.045" /> <!-- Mass of sensor    -->
+  <property name="mass_usound"      value="0.100" /> <!-- Mass of sensor    -->
   <property name="base_x_origin_to_ultrasound_origin" value="0.45639" />
   <property name="base_y_origin_to_ultrasound_origin" value="0.10000" />
@@ -38,11 +38,7 @@
     </link>
     <gazebo reference="${fb}_${cnc}_${lr}_ultrasound">
-      <mu1 value="1.0"/>
-      <mu2 value="1.0"/>
-      <kp  value="10000000.0" />
-      <kd  value="1.0" />
-      <fdir1 value="1 0 0"/>
-      <material>Gazebo/Grey</material>
-      <turnGravityOff>false</turnGravityOff>
+      <static>true</static>
+      <material>Gazebo/Blue</material>
+      <turnGravityOff>true</turnGravityOff>
     </gazebo>
     <joint name="${fb}_${cnc}_${lr}_ultrasound_joint" type="fixed">
@@ -51,15 +47,4 @@
       <origin xyz="${translateX * base_x_origin_to_ultrasound_origin} ${translateY * base_y_origin_to_ultrasound_origin} ${base_z_origin_to_ultrasound_origin + translateZ}" rpy="0 0 ${rotateTheta*Pi/180}"/>
     </joint>
-    <!-- Transmission is important to link the joints and the controller -->
-    <transmission name="${fb}_${cnc}_${lr}_ultrasound_joint_trans">
-      <type>transmission_interface/SimpleTransmission</type>
-      <joint name="${fb}_${cnc}_${lr}_ultrasound_joint">
-        <hardwareInterface>EffortJointInterface</hardwareInterface>
-      </joint>
-      <actuator name="${fb}_${cnc}_${lr}_ultrasound_joint_motor">
-        <hardwareInterface>EffortJointInterface</hardwareInterface>
-        <mechanicalReduction>1</mechanicalReduction>
-      </actuator>
-    </transmission>
   </xacro:macro>
 </robot>

Commit message: Updating gazebo frames

File: src/raskar_urdf/urdf/lidar.urdf.xacro (robot description, xacro)
@@ -30,5 +30,5 @@
       <inertial>
         <mass value="${mass_lidar}" />
-        <origin xyz="0 0 0" />
+        <origin xyz="0 0 0"/>
         <cylinder_inertia  m="${mass_lidar}" r="${diam_lidar/2}" h="${thickness_lidar}" />
       </inertial>

Commit message: Update lidar.urdf.xacro

File: src/raskar_urdf/urdf/lidar.urdf.xacro (robot description, xacro)
@@ -46,5 +46,5 @@
       <parent link="${parent}"/>
       <child link="${fb}_${cnc}_${lrc}_lidar"/>
-      <origin xyz="${translateX * base_x_origin_to_lidar_origin} ${translateY * base_y_origin_to_lidar_origin} ${translateZ * base_z_origin_to_lidar_origin + (thickness_lidar/2)}" rpy="0 0 0" />
+      <origin xyz="${translateX * base_x_origin_to_lidar_origin} ${translateY * base_y_origin_to_lidar_origin} ${base_z_origin_to_lidar_origin + (thickness_lidar/2) + translateZ}" rpy="0 0 0" />
     </joint>
     <!-- Transmission is important to link the joints and the controller -->

Commit message: Updating move_base_simple

File: src/raskar_urdf/urdf/lidar.urdf.xacro (robot description, xacro)
@@ -30,16 +30,12 @@
       <inertial>
         <mass value="${mass_lidar}" />
-        <origin xyz="0 0 0" />
+        <origin xyz="0 0 0"/>
         <cylinder_inertia  m="${mass_lidar}" r="${diam_lidar/2}" h="${thickness_lidar}" />
       </inertial>
     </link>
     <gazebo reference="${fb}_${cnc}_${lrc}_lidar">
-      <mu1 value="1.0"/>
-      <mu2 value="1.0"/>
-      <kp  value="10000000.0" />
-      <kd  value="1.0" />
-      <fdir1 value="1 0 0"/>
-      <material>Gazebo/Grey</material>
-      <turnGravityOff>false</turnGravityOff>
+      <static>true</static>
+      <material>Gazebo/Black</material>
+      <turnGravityOff>true</turnGravityOff>
     </gazebo>
     <joint name="${fb}_${cnc}_${lrc}_lidar_joint" type="fixed">
@@ -48,15 +44,4 @@
       <origin xyz="${translateX * base_x_origin_to_lidar_origin} ${translateY * base_y_origin_to_lidar_origin} ${base_z_origin_to_lidar_origin + (thickness_lidar/2) + translateZ}" rpy="0 0 0" />
     </joint>
-    <!-- Transmission is important to link the joints and the controller -->
-    <transmission name="${fb}_${cnc}_${lrc}_lidar_joint_trans">
-      <type>transmission_interface/SimpleTransmission</type>
-      <joint name="${fb}_${cnc}_${lrc}_lidar_joint">
-        <hardwareInterface>EffortJointInterface</hardwareInterface>
-      </joint>
-      <actuator name="${fb}_${cnc}_${lrc}_lidar_joint_motor">
-        <hardwareInterface>EffortJointInterface</hardwareInterface>
-        <mechanicalReduction>1</mechanicalReduction>
-      </actuator>
-    </transmission>
   </xacro:macro>
 </robot>

File: src/raskar_urdf/urdf/raskar_gazebo.xacro (robot description, xacro)
@@ -14,4 +14,6 @@
   <xacro:property name="thickness_lidar" value="0.045" /> <!-- Thickness of wheel -->
   <xacro:property name="safety_offset"   value="1.25"  /> <!-- Percentage safety  -->
+  <xacro:property name="floor_clearance" value="0.0350"/> <!-- Floor clearance    -->
+  <xacro:property name="model_offset"    value="0.0127"/> <!-- Floor clearance    -->
   <!-- Gazebo initializer -->
   <!-- Import all Gazebo-customization elements, including Gazebo colors -->
@@ -24,4 +26,5 @@
   <!-- Import Sensors -->
   <xacro:include filename="$(find raskar_urdf)/urdf/ultrasound.urdf.xacro" />
+  <xacro:include filename="$(find raskar_urdf)/urdf/lidar.urdf.xacro" />
   <!-- Macro for calculating inertia of cylinder -->
   <macro name="cylinder_inertia" params="m r h">
@@ -30,8 +33,14 @@
               izz="${m*r*r/2}" />
   </macro>
+  <!-- Macro for calculating inertia of box -->
+  <macro name="box_inertia" params="m h l w">
+    <inertia  ixx="${m*(h*h+l*l)/12}" ixy = "0" ixz = "0"
+              iyy="${m*(w*w+l*l)/12}" iyz = "0"
+              izz="${m*(w*w+h*h)/12}" />
+  </macro>
   <!-- Used for fixing robot to Gazebo -->
-  <!-- link name="world"/>
+  <!-- link name="floor"/>
   <joint name="fixed" type="fixed">
-    <parent link="world"/>
+    <parent link="floor"/>
     <child link="base_footprint"/>
   </joint -->
@@ -39,5 +48,5 @@
   <!-- base_footprint is a fictitious link(frame) that is on the ground right below base_link origin -->
   <link name="base_footprint">
-    <inertial>
+    <!-- inertial>
       <mass value="0.0001" />
       <origin xyz="0 0 0" />
@@ -45,5 +54,5 @@
           iyy="0.0001" iyz="0.0"
           izz="0.0001" />
-    </inertial>
+    </inertial -->
     <visual>
         <origin xyz="0 0 0" rpy="0 0 0" />
@@ -57,5 +66,5 @@
   </gazebo>
   <joint name="base_footprint_joint" type="fixed">
-    <origin xyz="0 0 0" rpy="0 0 0" />
+    <origin xyz="0 0 ${height_body/2}" rpy="0 0 0" />
     <parent link="base_footprint"/>
     <child link="base_link" />
@@ -64,5 +73,5 @@
   <link name="base_link">
     <visual>
-      <origin rpy="1.571 0 0" xyz="0 0 -0.0127"/> <!-- Half an inch due to different wheels set up -->
+      <origin rpy="1.571 0 0" xyz="0 0 ${-height_body/2-floor_clearance-model_offset}"/> <!-- Half an inch due to different wheels set up -->
       <geometry>
         <mesh filename="package://raskar_urdf/meshes/body_parts.stl" scale="0.001 0.001 0.001" />
@@ -78,11 +87,10 @@
     </collision>
     <inertial>
-      <mass value="${mass_wheel}"/>
-      <inertia
-	  ixx="${mass_body / 12.0 * (height_body*height_body + length_body*length_body)}" ixy="0.0" ixz="0.0"
-	  iyy="${mass_body / 12.0 * (width_body*width_body + length_body*length_body)}" iyz="0.0"
-	  izz="${mass_body / 12.0 * (width_body*width_body + height_body*height_body)}"/>
+      <mass value="${mass_body}"/>
+      <origin xyz="0 0 0" />
+      <box_inertia  m="${mass_body}" h="${height_body}" l="${length_body}" w="${width_body}" />
     </inertial>
   </link>
+<<<<<<< HEAD
   <!-- Wheels definition -->
   <wheel fb="bk" lr="right"  parent="base_link" translateX="-1" translateY="-1" translateZ="1" flipY="1"/>
@@ -92,11 +100,20 @@
   <!-- Lidar definition -->
   <lidar fb="fr"  cnc="nocorner"   lrc="center"   parent="base_link" translateX="1" translateY="1"  translateZ="1" flipX="0" flipY="0" flipZ="0"/>
-  <!-- Ultrasound sensors Definitions -->
-  <ultrasound fb="front" cnc="nocorner" lr="right"  parent="base_link" translateX="1" translateY="-1" translateZ="1" flipX="90" flipY="0" flipZ="90"/>
-  <ultrasound fb="front" cnc="nocorner" lr="left"   parent="base_link" translateX="1" translateY="1"  translateZ="1" flipX="90" flipY="0" flipZ="90"/>
-  <ultrasound fb="front" cnc="corner"   lr="right"  parent="base_link" translateX="0.8991870987"  translateY="-2.5038" translateZ="1" flipX="90" flipY="0" flipZ="45"/>
-  <ultrasound fb="front" cnc="corner"   lr="left"   parent="base_link" translateX="0.8991870987"  translateY="2.5038"  translateZ="1" flipX="90" flipY="0" flipZ="135"/>
-  <ultrasound fb="back"  cnc="corner"   lr="right"  parent="base_link" translateX="-0.8991870987" translateY="-2.5038" translateZ="1" flipX="90" flipY="0" flipZ="315"/>
-  <ultrasound fb="back"  cnc="corner"   lr="left"   parent="base_link" translateX="-0.8991870987" translateY="2.5038"  translateZ="1" flipX="90" flipY="0" flipZ="225"/>
+=======
+  <!-- Wheels Definition -->
+  <wheel fb="bk" lr="right"  parent="base_link" translateX="-1" translateY="-1" translateZ="${((-height_body/2)-floor_clearance)}" flipY="1"/>
+  <wheel fb="fr" lr="right"  parent="base_link" translateX="1"  translateY="-1" translateZ="${((-height_body/2)-floor_clearance)}" flipY="1"/>
+  <wheel fb="fr" lr="left" parent="base_link" translateX="1"  translateY="1"  translateZ="${((-height_body/2)-floor_clearance)}" flipY="1"/>
+  <wheel fb="bk" lr="left" parent="base_link" translateX="-1" translateY="1"  translateZ="${((-height_body/2)-floor_clearance)}" flipY="1"/>
+>>>>>>> b2afef46d33e9755fd909ccf55dd974d8138fe6e
+  <!-- Ultrasound sensors definition -->
+  <ultrasound fb="fr" cnc="nocorner" lr="right"  parent="base_link" translateX="1" translateY="-1" translateZ="${((-height_body/2)-floor_clearance)}" flipX="90" flipY="0" flipZ="90" rotateTheta="0"/>
+  <ultrasound fb="fr" cnc="nocorner" lr="left"   parent="base_link" translateX="1" translateY="1"  translateZ="${((-height_body/2)-floor_clearance)}" flipX="90" flipY="0" flipZ="90" rotateTheta="0"/>
+  <ultrasound fb="fr" cnc="corner"   lr="right"  parent="base_link" translateX="0.8991870987"  translateY="-2.5038" translateZ="${((-height_body/2)-floor_clearance)}" flipX="90" flipY="0" flipZ="90" rotateTheta="-45"/>
+  <ultrasound fb="fr" cnc="corner"   lr="left"   parent="base_link" translateX="0.8991870987"  translateY="2.5038"  translateZ="${((-height_body/2)-floor_clearance)}" flipX="90" flipY="0" flipZ="90" rotateTheta="45"/>
+  <ultrasound fb="bk" cnc="corner"   lr="right"  parent="base_link" translateX="-0.8991870987" translateY="-2.5038" translateZ="${((-height_body/2)-floor_clearance)}" flipX="90" flipY="0" flipZ="90" rotateTheta="225"/>
+  <ultrasound fb="bk" cnc="corner"   lr="left"   parent="base_link" translateX="-0.8991870987" translateY="2.5038"  translateZ="${((-height_body/2)-floor_clearance)}" flipX="90" flipY="0" flipZ="90" rotateTheta="135"/>
+  <!-- Lidar definition -->
+  <lidar fb="fr"  cnc="nocorner"   lrc="center"  parent="base_link" translateX="1" translateY="1"  translateZ="${(-height_body/2)-floor_clearance}" flipX="0" flipY="0" flipZ="0"/>
   <!-- Motion controller -->
   <!-- Planar drive controller  -->

File: src/raskar_urdf/urdf/raskar_rviz.xacro (robot description, xacro)
@@ -17,4 +17,7 @@
   <xacro:property name="floor_clearance" value="0.0350"/> <!-- Floor clearance    -->
   <xacro:property name="model_offset"    value="0.0127"/> <!-- Floor clearance    -->
+<<<<<<< HEAD
+=======
+>>>>>>> b2afef46d33e9755fd909ccf55dd974d8138fe6e
   <!-- Gazebo initializer -->
   <!-- Import all Gazebo-customization elements, including Gazebo colors -->
@@ -28,5 +31,5 @@
   <xacro:include filename="$(find raskar_urdf)/urdf/ultrasound.urdf.xacro" />
   <xacro:include filename="$(find raskar_urdf)/urdf/lidar.urdf.xacro" />
-  <!-- Used for fixing robot to Gazebo -->
+   <!-- Used for fixing robot to Gazebo -->
   <link name="world"/>
   <joint name="fixed" type="fixed">

Commit message: Including pub, sub object for laser scanner

File: src/raskar_urdf/urdf/lidar.urdf.xacro (robot description, xacro)
@@ -16,5 +16,5 @@
     <link name="${fb}_${cnc}_${lrc}_lidar">
       <visual>
-        <origin xyz="0 0 0" rpy="${flipX*Pi/180} ${flipY*Pi/180} ${flipZ*Pi/180}"/>
+        <origin xyz="0 0 0" rpy="0 0 0"/>
         <geometry>
           <cylinder length="${thickness_lidar}" radius="${diam_lidar/2}" />
@@ -42,5 +42,5 @@
       <parent link="${parent}"/>
       <child link="${fb}_${cnc}_${lrc}_lidar"/>
-      <origin xyz="${translateX * base_x_origin_to_lidar_origin} ${translateY * base_y_origin_to_lidar_origin} ${base_z_origin_to_lidar_origin + (thickness_lidar/2) + translateZ}" rpy="0 0 0" />
+      <origin xyz="${translateX * base_x_origin_to_lidar_origin} ${translateY * base_y_origin_to_lidar_origin} ${base_z_origin_to_lidar_origin + (thickness_lidar/2) + translateZ}" rpy="${flipX*Pi/180} ${flipY*Pi/180} ${flipZ*Pi/180}" />
     </joint>
   </xacro:macro>

File: src/raskar_urdf/urdf/raskar_gazebo.xacro (robot description, xacro)
@@ -105,5 +105,5 @@
   <ultrasound fb="bk" cnc="corner"   lr="left"   parent="base_link" translateX="-0.8991870987" translateY="2.5038"  translateZ="${((-height_body/2)-floor_clearance)}" flipX="90" flipY="0" flipZ="90" rotateTheta="135"/>
   <!-- Lidar definition -->
-  <lidar fb="fr"  cnc="nocorner"   lrc="center"  parent="base_link" translateX="1" translateY="1"  translateZ="${(-height_body/2)-floor_clearance}" flipX="0" flipY="0" flipZ="0"/>
+  <lidar fb="fr"  cnc="nocorner"   lrc="center"  parent="base_link" translateX="1" translateY="1"  translateZ="${(-height_body/2)-floor_clearance}" flipX="0" flipY="0" flipZ="180"/>
   <!-- Motion controller -->
   <!-- Planar drive controller  -->
