Commit message: Adding initial navigation files and fake laser sensor information from gazebo

File: src/raskar_urdf/urdf/lidar.urdf.xacro (robot description, xacro)
@@ -35,7 +35,7 @@
     </link>
     <gazebo reference="${fb}_${cnc}_${lrc}_lidar">
-      <static>true</static>
+      <!-- static>true</static -->
       <material>Gazebo/Black</material>
-      <turnGravityOff>true</turnGravityOff>
+      <turnGravityOff>false</turnGravityOff>
     </gazebo>
     <joint name="${fb}_${cnc}_${lrc}_lidar_joint" type="fixed">

File: src/raskar_urdf/urdf/raskar_gazebo.xacro (robot description, xacro)
@@ -81,8 +81,9 @@
     </visual>
     <collision>
-      <origin rpy="0 0 0" xyz="0 0 0.25"/>
+      <origin rpy="1.571 0 0" xyz="0 0 ${-height_body/2-floor_clearance-model_offset}"/>
       <geometry>
         <!--box size="0.948 0.636 0.3"/-->
-        <box size="0.998 0.678 0.35"/>
+        <!--box size="0.998 0.678 0.35"/-->
+        <mesh filename="package://raskar_urdf/meshes/body_parts.stl" scale="0.001 0.001 0.001" />
       </geometry>
     </collision>
