Commit message: Update wheel.urdf.xacro

File: src/raskar_urdf/urdf/wheel.urdf.xacro (robot description, xacro)
@@ -48,5 +48,5 @@
       <parent link="${parent}"/>
       <child link="${fb}_${lr}_wheel"/>
-      <origin xyz="${translateX * base_x_origin_to_wheel_origin} ${translateY * base_y_origin_to_wheel_origin} ${translateZ * base_z_origin_to_wheel_origin}" rpy="0 0 0" />
+      <origin xyz="${translateX * base_x_origin_to_wheel_origin} ${translateY * base_y_origin_to_wheel_origin} ${base_z_origin_to_wheel_origin + translateZ}" rpy="0 0 0" />
       <axis xyz="0 1 0" rpy="0  0" />
       <limit effort="100" velocity="100"/>

Commit message: Config modified

File: src/raskar_urdf/urdf/wheel.urdf.xacro (robot description, xacro)
@@ -18,6 +18,6 @@
         <origin xyz="0 0 0" rpy="${flipY*Pi/2} 0  0 " />
         <geometry>
-          <!-- cylinder length="${thickness_wheel}" radius="${diam_wheel/2}" /-->
-          <mesh filename="package://raskar_urdf/meshes/5_in_mecanum.stl" scale="0.001 0.001 0.001" />
+          < cylinder length="${thickness_wheel}" radius="${diam_wheel/2}" />
+          <!-- mesh filename="package://raskar_urdf/meshes/5_in_mecanum.stl"  scale="0.001 0.001 0.001" /-->
         </geometry>
         <material name="dark_yellow" />
